Commit message: Fixed TCP_link missing collision geometry

File: kuka_waam_description/urdf/welding_torch.urdf.xacro (robot description, xacro)
@@ -98,4 +98,5 @@
       <child link="${prefix}tcp_link"/>
     </joint>
+    <!-- FIX: Added collision geometry to tcp_link -->
     <link name="${prefix}tcp_link">
       <visual>
@@ -108,4 +109,17 @@
         </material>
       </visual>
+      <collision>
+        <origin xyz="0 0 0" rpy="0 0 0"/>
+        <geometry>
+          <sphere radius="0.005"/>
+        </geometry>
+      </collision>
+      <inertial>
+        <origin xyz="0 0 0" rpy="0 0 0"/>
+        <mass value="0.001"/>
+        <inertia ixx="0.000001" ixy="0" ixz="0"
+                 iyy="0.000001" iyz="0"
+                 izz="0.000001"/>
+      </inertial>
     </link>
     <!-- Gas nozzle -->
