Commit message: _a to _

File: kuka_waam_description/urdf/kr6_r900_waam.urdf.xacro (robot description, xacro)
@@ -1,5 +1,5 @@
 <?xml version="1.0"?>
 <robot xmlns:xacro="http://www.ros.org/wiki/xacro" name="kr6_r900_waam">
-  <!-- Include base robot -->
+  <!-- Include base robot macro -->
   <xacro:include filename="$(find kuka_agilus_support)/urdf/kr6_r900_sixx_macro.xacro"/>
   <!-- Include welding torch -->
@@ -9,37 +9,67 @@
   <xacro:arg name="mode" default="mock"/>
   <xacro:arg name="use_fake_hardware" default="true"/>
-  <!-- World frame -->
-  <link name="world"/>
   <!-- Instantiate robot -->
-  <xacro:kr6_r900_sixx
+  <xacro:kuka_kr6_r900_sixx_robot
     prefix="$(arg prefix)"
-    mode="$(arg mode)"
-    use_fake_hardware="$(arg use_fake_hardware)">
+    package_name="kuka_agilus_support">
     <origin xyz="0 0 0" rpy="0 0 0"/>
-  </xacro:kr6_r900_sixx>
-  <!-- Fixed joint from world to robot base -->
-  <joint name="world_to_base_joint" type="fixed">
-    <origin xyz="0 0 0" rpy="0 0 0"/>
-    <parent link="world"/>
-    <child link="$(arg prefix)base_link"/>
-  </joint>
+  </xacro:kuka_kr6_r900_sixx_robot>
   <!-- Attach welding torch to flange -->
   <xacro:welding_torch prefix="$(arg prefix)" parent_link="$(arg prefix)flange">
     <origin xyz="0 0 0" rpy="0 0 0"/>
   </xacro:welding_torch>
-  <!-- Update tool0 to be at TCP -->
-  <joint name="$(arg prefix)flange_to_tool0" type="fixed">
-    <origin xyz="0 0 0.232" rpy="0 0 0"/>  <!-- Height to TCP -->
-    <parent link="$(arg prefix)flange"/>
-    <child link="$(arg prefix)tool0"/>
-  </joint>
+  <!-- ADD THIS: ros2_control configuration -->
+  <ros2_control name="kuka_waam_system" type="system">
+    <hardware>
+      <xacro:if value="$(arg use_fake_hardware)">
+        <plugin>mock_components/GenericSystem</plugin>
+      </xacro:if>
+      <xacro:unless value="$(arg use_fake_hardware)">
+        <plugin>kuka_rsi_hardware_interface/KukaRSIHardwareInterface</plugin>
+      </xacro:unless>
+    </hardware>
+    <!-- Joint 1 -->
+    <joint name="$(arg prefix)joint_1">
+      <command_interface name="position"/>
+      <state_interface name="position"/>
+      <state_interface name="velocity"/>
+    </joint>
+    <!-- Joint 2 -->
+    <joint name="$(arg prefix)joint_2">
+      <command_interface name="position"/>
+      <state_interface name="position"/>
+      <state_interface name="velocity"/>
+    </joint>
+    <!-- Joint 3 -->
+    <joint name="$(arg prefix)joint_3">
+      <command_interface name="position"/>
+      <state_interface name="position"/>
+      <state_interface name="velocity"/>
+    </joint>
+    <!-- Joint 4 -->
+    <joint name="$(arg prefix)joint_4">
+      <command_interface name="position"/>
+      <state_interface name="position"/>
+      <state_interface name="velocity"/>
+    </joint>
+    <!-- Joint 5 -->
+    <joint name="$(arg prefix)joint_5">
+      <command_interface name="position"/>
+      <state_interface name="position"/>
+      <state_interface name="velocity"/>
+    </joint>
+    <!-- Joint 6 -->
+    <joint name="$(arg prefix)joint_6">
+      <command_interface name="position"/>
+      <state_interface name="position"/>
+      <state_interface name="velocity"/>
+    </joint>
+  </ros2_control>
   <!-- Gazebo plugins -->
-  <xacro:if value="$(arg use_fake_hardware)">
-    <gazebo>
-      <plugin filename="libgazebo_ros2_control.so" name="gazebo_ros2_control">
-        <parameters>$(find kuka_waam_description)/config/ros2_controllers.yaml</parameters>
-      </plugin>
-    </gazebo>
-  </xacro:if>
+  <gazebo>
+    <plugin filename="libign_ros2_control-system" name="ign_ros2_control::IgnitionROS2ControlPlugin">
+      <parameters>$(find kuka_waam_description)/config/ros2_controllers.yaml</parameters>
+    </plugin>
+  </gazebo>
   <!-- Welding torch Gazebo properties -->
   <gazebo reference="$(arg prefix)torch_body_link">
@@ -52,12 +82,3 @@
     <material>Gazebo/Red</material>
   </gazebo>
-  <!-- Optional: Welding effect plugin -->
-  <gazebo>
-    <plugin name="welding_torch_plugin" filename="libwelding_torch_plugin.so">
-      <arc_topic>/welding_state</arc_topic>
-      <tcp_link>$(arg prefix)tcp_link</tcp_link>
-      <heat_radius>0.01</heat_radius>
-      <heat_intensity>1000.0</heat_intensity>
-    </plugin>
-  </gazebo>
 </robot>

Commit message: created a default rviz that's responsive

File: kuka_waam_description/urdf/kr6_r900_waam.urdf.xacro (robot description, xacro)
@@ -17,5 +17,5 @@
   <!-- Attach welding torch to flange -->
   <xacro:welding_torch prefix="$(arg prefix)" parent_link="$(arg prefix)flange">
-    <origin xyz="0 0 0" rpy="0 0 0"/>
+    <origin xyz="0 0 0" rpy="0 1.57 0"/>
   </xacro:welding_torch>
   <!-- ADD THIS: ros2_control configuration -->

Commit message: getting the welding torch to work

File: kuka_waam_description/urdf/kr6_r900_waam.urdf.xacro (robot description, xacro)
@@ -76,8 +76,8 @@
     <material>Gazebo/Blue</material>
   </gazebo>
-  <gazebo reference="$(arg prefix)contact_tip_link">
+  <!-- <gazebo reference="$(arg prefix)contact_tip_link">
     <material>Gazebo/Orange</material>
-  </gazebo>
-  <gazebo reference="$(arg prefix)tcp_link">
+  </gazebo> -->
+  <gazebo reference="$(arg prefix)gas_nozzle_link">
     <material>Gazebo/Red</material>
   </gazebo>

File: kuka_waam_description/urdf/welding_torch.urdf.xacro (robot description, xacro)
@@ -32,5 +32,5 @@
       </inertial>
     </link>
-    <!-- Torch body -->
+    <!-- Torch body - UPDATED TO USE STL MESH -->
     <joint name="${prefix}torch_body_joint" type="fixed">
       <origin xyz="0 0 0.05" rpy="0 0 0"/>
@@ -39,8 +39,9 @@
     </joint>
     <link name="${prefix}torch_body_link">
+      <!-- Visual: Use STL mesh -->
       <visual>
-        <origin xyz="0 0 0.075" rpy="0 0 0"/>
+        <origin xyz="0 0 0.05" rpy="1.5708  3.1416  1.5708"/>
         <geometry>
-          <cylinder radius="0.025" length="0.15"/>
+          <mesh filename="package://kuka_waam_description/meshes/welding_torch/torch_body.stl" scale="0.001 0.001 0.001"/>
         </geometry>
         <material name="blue">
@@ -49,7 +50,7 @@
       </visual>
       <collision>
-        <origin xyz="0 0 0.075" rpy="0 0 0"/>
+        <origin xyz="0 0 0.05" rpy="1.5708  3.1416 1.5708"/>
         <geometry>
-          <cylinder radius="0.025" length="0.15"/>
+          <mesh filename="package://kuka_waam_description/meshes/welding_torch/torch_body.stl" scale="0.001 0.001 0.001"/>
         </geometry>
       </collision>
@@ -63,5 +64,5 @@
     </link>
     <!-- Contact tip (welding wire exit point) -->
-    <joint name="${prefix}contact_tip_joint" type="fixed">
+    <!-- <joint name="${prefix}contact_tip_joint" type="fixed">
       <origin xyz="0 0 0.15" rpy="0 0 0"/>
       <parent link="${prefix}torch_body_link"/>
@@ -92,11 +93,10 @@
       </inertial>
     </link>
-    <!-- TCP (Tool Center Point) - wire stick-out point -->
     <joint name="${prefix}tcp_joint" type="fixed">
       <origin xyz="0 0 0.032" rpy="0 0 0"/>
       <parent link="${prefix}contact_tip_link"/>
       <child link="${prefix}tcp_link"/>
-    </joint>
-    <!-- FIX: Added collision geometry to tcp_link -->
+    </joint> -->
+<!--
     <link name="${prefix}tcp_link">
       <visual>
@@ -122,16 +122,17 @@
                  izz="0.000001"/>
       </inertial>
-    </link>
-    <!-- Gas nozzle -->
+    </link> -->
+    <!-- Gas nozzle - UPDATED TO USE STL MESH -->
     <joint name="${prefix}gas_nozzle_joint" type="fixed">
-      <origin xyz="0 0 0.0" rpy="0 0 0"/>
+      <origin xyz="0 0 0" rpy="0 0 0"/>
       <parent link="${prefix}torch_body_link"/>
       <child link="${prefix}gas_nozzle_link"/>
     </joint>
     <link name="${prefix}gas_nozzle_link">
+      <!-- Visual: Use STL mesh -->
       <visual>
-        <origin xyz="0 0 0.11" rpy="0 0 0"/>
+        <origin xyz="0 0 0.05" rpy="1.5708  3.1416  1.5708"/>
         <geometry>
-          <cylinder radius="0.035" length="0.08"/>
+          <mesh filename="package://kuka_waam_description/meshes/welding_torch/nozzle.stl" scale="0.001 0.001 0.001"/>
         </geometry>
         <material name="light_grey">
@@ -140,7 +141,7 @@
       </visual>
       <collision>
-        <origin xyz="0 0 0.11" rpy="0 0 0"/>
+        <origin xyz="0 0 0.05" rpy="1.5708  3.1416  1.5708"/>
         <geometry>
-          <cylinder radius="0.035" length="0.08"/>
+          <mesh filename="package://kuka_waam_description/meshes/welding_torch/nozzle.stl" scale="0.001 0.001 0.001"/>
         </geometry>
       </collision>
